Commit message: python script to calculate inertia tensor or updated README.md

File: gripper.urdf (robot description, URDF)
Before this commit: robot gripper, 6 links, 5 joints
Links:
- link base_link: mass None -> 0.0; geometry collision cylinder length=0.006 radius=0.039; visual cylinder length=0.006 radius=0.039
- link first_link: mass None -> 0.0; geometry collision box size=0.08 0.06 0.069; visual box size=0.08 0.06 0.069
- link left_finger: mass None -> 0.0; geometry collision box size=0.01 0.01 0.035; visual box size=0.01 0.01 0.035
- link left_finger_base: mass None -> 0.0; geometry collision box size=0.03 0.01 0.008; visual box size=0.03 0.01 0.008
- link right_finger: mass None -> 0.0; geometry collision box size=0.01 0.01 0.035; visual box size=0.01 0.01 0.035
- link right_finger_base: mass None -> 0.0; geometry collision box size=0.025 0.01 0.008; visual box size=0.025 0.01 0.008

Commit message: updated urdf to be more precise with gripper, updated tensor_interia.py, updated readme.md and added img

File: gripper.urdf (robot description, URDF)
Before this commit: robot gripper, 6 links, 5 joints
Links:
- link first_link: geometry collision box size=0.08 0.06 0.069; visual box size=0.08 0.06 0.063
- link left_finger: geometry collision box size=0.01 0.01 0.034; visual box size=0.01 0.01 0.034
- link left_finger_base: geometry collision box size=0.025 0.005 0.008; visual box size=0.025 0.005 0.008
- link right_finger: geometry collision box size=0.01 0.01 0.034; visual box size=0.01 0.01 0.034
- link right_finger_base: geometry collision box size=0.025 0.005 0.008; visual box size=0.025 0.005 0.008
Joints:
- joint gripper_base: origin xyz=0 0 0.003 -> xyz=0 0 0.006
- joint left_finger_base_joint: axis 0 0 0 -> -1 0 0; limit (none) -> lower=0.0 upper=0.03 effort=300 velocity=2.0; origin xyz=0.0 0.0 0.069 -> xyz=0.0 0.0 0.063; type fixed -> prismatic
- joint left_finger_joint: axis -1 0 0 -> 0 0 0; limit lower=0.0 upper=0.03 effort=300 velocity=2.0 -> (none); origin xyz=0 0 0.005 rpy=0 0 0 -> xyz=0 0 0.008 rpy=0 0 0; type prismatic -> fixed
- joint right_finger_base_joint: axis 0 0 0 -> 1 0 0; limit (none) -> lower=0.0 upper=0.03 effort=300 velocity=2.0; origin xyz=0 0 0.069 -> xyz=0 0 0.063; type fixed -> prismatic
- joint right_finger_joint: axis 1 0 0 -> 0 0 0; limit lower=0.0 upper=0.03 effort=300 velocity=2.0 -> (none); origin xyz=0 0 0.005 rpy=0 0 0 -> xyz=0 0 0.008 rpy=0 0 0; type prismatic -> fixed

Commit message: updated link names

File: gripper.urdf (robot description, URDF)
Before this commit: robot gripper, 6 links, 5 joints
Links:
- removed link base_link
- removed link first_link
- added link gripper_base_link, mass 0.0; collision cylinder length=0.006 radius=0.039; visual cylinder length=0.006 radius=0.039
- added link gripper_first_link, mass 0.0; collision box size=0.08 0.06 0.069; visual box size=0.08 0.06 0.063
Joints:
- joint gripper_base: child first_link -> gripper_first_link; parent base_link -> gripper_base_link
- joint left_finger_base_joint: parent first_link -> gripper_first_link
- joint right_finger_base_joint: parent first_link -> gripper_first_link

Commit message: control xacros added

File: gripper.urdf (robot description, URDF)
Before this commit: robot gripper, 6 links, 5 joints
Joints:
- joint left_finger_base_joint: mimic (none) -> joint=right_finger_base_joint multiplier=1 offset=0
