Commit message: modified mass values innertia tag and modified xacro files

File: gripper.macro.xacro (robot description, xacro)
@@ -1,8 +1,16 @@
 <?xml version="1.0"?>
 <robot xmlns:xacro="http://www.ros.org/wiki/xacro"
-       name="igus_rebel_6dof" >
+       name="gripper" >
   <!-- Include all igus_rebel_6dof macros -->
   <!-- this is designed to be put together inside irc_ros_description packges. change package name as required -->
-  <xacro:include filename="$(find irc_ros_description)/urdf/end_effector/gripper.xacro" />
-  <xacro:include filename="$(find irc_ros_description)/urdf/end_effector/gripper.ros2_control.xacro" />
+  <xacro:include filename="$(find irc_ros_description)/urdf/grippers/gripper.urdf" />
+  <xacro:include filename="$(find irc_ros_description)/urdf/grippers/gripper.ros2_control.xacro" />
+  <xacro:macro name="gripper" params="parent_link hardware_protocol is_ignition">
+    <xacro:gripper_controller hardware_protocol="${hardware_protocol}" is_ignition="${is_ignition}" />
+    <joint name="gripper_world_base" type="fixed">
+      <parent link="flange"/>
+      <child link="gripper_base_link"/>
+      <origin xyz="0 0 0" rpy="0.0 1.57 0.0"/>
+  </joint>
+  </xacro:macro>
 </robot>

File: gripper.ros2_control.xacro (robot description, xacro)
@@ -1,5 +1,5 @@
 <?xml version="1.0" ?>
 <robot xmlns:xacro="http://www.ros.org/wiki/xacro">
-  <xacro:macro name="igus_rebel_6dof_01_ros2_control" params="hardware_protocol is_ignition">
+  <xacro:macro name="gripper_controller" params="hardware_protocol is_ignition">
     <ros2_control name="igus_rebel_6dof" type="system">
       <hardware>

File: gripper.urdf (robot description, URDF)
Before this commit: robot gripper, 6 links, 5 joints
Links:
- link gripper_base_link: mass 0.0 -> 0.04
- link gripper_first_link: mass 0.0 -> 0.32
- link left_finger: mass 0.0 -> 0.015
- link left_finger_base: mass 0.0 -> 0.005
- link right_finger: mass 0.0 -> 0.015
- link right_finger_base: mass 0.0 -> 0.005
